Commit message: generate map using slam toolbox Load the map Get the initial position using AMCL
Note:
- Haven't build the navigation for the robot
- Haven't control the robot by using joystick
- Haven't build the web app for the robot after control by gamepad

Signed-off-by: VuongAdonis <vuong03062003@gmail.com>

File: src/my_bot/description/robot.urdf.xacro (robot description, xacro)
@@ -4,5 +4,5 @@
     <xacro:include filename="lidar.xacro" />
     <xacro:include filename="camera.xacro" />
-    <!-- <xacro:include filename="gazebo_control.xacro"/> -->
-    <xacro:include filename="ros2_control.xacro"/>
+    <xacro:include filename="gazebo_control.xacro"/>
+    <!-- <xacro:include filename="ros2_control.xacro"/> -->
 </robot>

File: src/my_bot/description/robot_core.xacro (robot description, xacro)
@@ -19,4 +19,12 @@
     <!-- BASE LINK -->
     <link name="base_link">
+    </link>
+    <!-- BASE_FOOTPRINT LINK-->
+    <joint name="base_footprint_join" type="fixed">
+        <parent link="base_link"/>
+        <child link="base_footprint"/>
+        <origin xyz="0 0 0" rpy="0 0 0"/>
+    </joint>
+    <link name="base_footprint">
     </link>
     <!-- CHASSIS LINK -->
